File: StandaloneLeakDetector.kicad_sch (KiCad schematic)
At the start: 12 parts, among them J1 TSW-102-07-L-S, J2 TSW-102-07-L-S, J3 Header, U1 QS6J11TR

Commit message: Remove imported symbol table fields
Parts:
- BT1: ALTIUM_VALUE * -> (none); AVAILABILITY In Stock -> (none); CHECK_PRICES https://www.snapeda.com/parts/BAT-HLD-005-THM/Linx/view-par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 -> (none); MF Linx Technologies Inc. -> (none); MP BAT-HLD-005-THM -> (none); PACKAGE None -> (none); PRICE None -> (none); PURCHASE-URL https://pricing.snapeda.com/search/part/BAT-HLD-005-THM/?re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 -> (none); Part Number (none) -> BAT-HLD-005-THM; SNAPEDA_LINK https://www.snapeda.com/parts/BAT-HLD-005-THM/Linx/view-par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 -> (none)
- D1: Part Number (none) -> SMTL6-RC
- D2: COPYRIGHT Copyright (C) 2022 Ultra Librarian. All rights reserved. -> (none); DIGI-KEY_PART_NUMBER_1 HLMP-EG15-UX000-ND -> (none); DIGI-KEY_PART_NUMBER_2 516-HLMP-EG15-UX000-ND -> (none); MANUFACTURER_PART_NUMBER HLMP-EG15-UX000 -> (none); MFR_NAME Avago Technologies -> (none); Part Number (none) -> HLMP-EG15-UX000; REFDES RefDes -> (none); TYPE DEV -> (none)
- J1, J2: COLOR Black -> (none); CONNECTOR TYPE Male Pin -> (none); CONTACT MATERIAL Bronze -> (none); CONTACT MATING LENGTH 0.23inch -> (none); CONTACT PLATING Gold -> (none); CONTACT TYPE Male Pin -> (none); CURRENT RATING 7.6A -> (none); DEPTH 2.54mm -> (none); GENDER Male -> (none); HOUSING COLOR Black -> (none); HOUSING MATERIAL Polyester -> (none); LEAD FREE Lead Free -> (none); LENGTH 5.08mm -> (none); MAX CURRENT RATING 7.6A -> (none); MAX OPERATING TEMPERATURE 125°C -> (none); MAX VOLTAGE RATING (AC) 550V -> (none); MIN OPERATING TEMPERATURE -55°C -> (none); MOUNT Through Hole -> (none); NUMBER OF CONTACTS 2 -> (none); NUMBER OF POSITIONS 2 -> (none); NUMBER OF ROWS 1 -> (none); ORIENTATION Straight -> (none); PACKAGE QUANTITY 1 -> (none); PACKAGING Bulk -> (none); PITCH 2.54mm -> (none); Part Number (none) -> TSW-102-07-L-S; RADIATION HARDENING No -> (none); REACH SVHC No SVHC -> (none); ROHS COMPLIANT Yes -> (none); SERIES TSW -> (none); TERMINATION Solder -> (none); VOLTAGE RATING 550V -> (none); WIDTH 2.54mm -> (none)
- R1: @ QTY 1500 -> (none); ALTIUM_VALUE 1M -> (none); COMPOSITION Thick Film -> (none); DATASHEETS http://industrial.panasonic.com/www-cgi/jvcr13pz.cgi?E+PZ+3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 -> (none); DIGI-KEY PART NUMBER P1.00MCCT-ND -> (none); FACTORY STOCK 0 -> (none); FAILURE RATE - -> (none); FEATURES Automotive AEC-Q200 -> (none); HEIGHT - SEATED (MAX) 0.028" (0.70mm) -> (none); IMAGE //media.digikey.com/Renders/Panasonic%20Renders/ERJ-0805%20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 -> (none); MANUFACTURER Panasonic Electronic Components -> (none); MINIMUM QUANTITY 1 -> (none); NUMBER OF TERMINATIONS 2 -> (none); OPERATING TEMPERATURE -55°C ~ 155°C -> (none); PACKAGE / CASE 0805 (2012 Metric) -> (none); PACKAGING Cut Tape (CT) -> (none); PART NUMBER ERJ-6ENF1004V -> (none); PART STATUS Active -> (none); POWER (WATTS) 0.125W, 1/8W -> (none); Part Number (none) -> ERJ-6ENF1004V; QUANTITY AVAILABLE 710452 -> (none); SERIES ERJ -> (none); SIZE / DIMENSION 0.079" L x 0.049" W (2.00mm x 1.25mm) -> (none); SUPPLIER DEVICE PACKAGE 0805 -> (none); TEMPERATURE COEFFICIENT ±100ppm/°C -> (none); TOLERANCE ±1% -> (none); UNIT PRICE (USD) 0.00729 -> (none)
- R2: @ QTY 1500 -> (none); ALTIUM_VALUE 10k -> (none); COMPOSITION Thick Film -> (none); DATASHEETS http://industrial.panasonic.com/www-cgi/jvcr13pz.cgi?E+PZ+3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 -> (none); DIGI-KEY PART NUMBER P10.0KCCT-ND -> (none); FACTORY STOCK 0 -> (none); FAILURE RATE - -> (none); FEATURES Automotive AEC-Q200 -> (none); HEIGHT - SEATED (MAX) 0.028" (0.70mm) -> (none); IMAGE //media.digikey.com/Renders/Panasonic%20Renders/ERJ-0805%20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 -> (none); MANUFACTURER Panasonic Electronic Components -> (none); MINIMUM QUANTITY 1 -> (none); NUMBER OF TERMINATIONS 2 -> (none); OPERATING TEMPERATURE -55°C ~ 155°C -> (none); PACKAGE / CASE 0805 (2012 Metric) -> (none); PACKAGING Cut Tape (CT) -> (none); PART NUMBER ERJ-6ENF1002V -> (none); PART STATUS Active -> (none); POWER (WATTS) 0.125W, 1/8W -> (none); Part Number (none) -> ERJ-6ENF1002V; QUANTITY AVAILABLE 3985614 -> (none); SERIES ERJ -> (none); SIZE / DIMENSION 0.079" L x 0.049" W (2.00mm x 1.25mm) -> (none); SUPPLIER DEVICE PACKAGE 0805 -> (none); TEMPERATURE COEFFICIENT ±100ppm/°C -> (none); TOLERANCE ±1% -> (none); UNIT PRICE (USD) 0.00729 -> (none)
- R3: @ QTY 1500 -> (none); ALTIUM_VALUE 20 -> (none); COMPOSITION Thick Film -> (none); DATASHEETS http://industrial.panasonic.com/www-cgi/jvcr13pz.cgi?E+PZ+3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 -> (none); DIGI-KEY PART NUMBER P20.0CCT-ND -> (none); FACTORY STOCK 0 -> (none); FAILURE RATE - -> (none); FEATURES Automotive AEC-Q200 -> (none); HEIGHT - SEATED (MAX) 0.028" (0.70mm) -> (none); IMAGE //media.digikey.com/Renders/Panasonic%20Renders/ERJ-0805%20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 -> (none); MANUFACTURER Panasonic Electronic Components -> (none); MINIMUM QUANTITY 1 -> (none); NUMBER OF TERMINATIONS 2 -> (none); OPERATING TEMPERATURE -55°C ~ 155°C -> (none); PACKAGE / CASE 0805 (2012 Metric) -> (none); PACKAGING Cut Tape (CT) -> (none); PART NUMBER ERJ-6ENF20R0V -> (none); PART STATUS Active -> (none); POWER (WATTS) 0.125W, 1/8W -> (none); Part Number (none) -> ERJ-6ENF20R0V; QUANTITY AVAILABLE 328732 -> (none); SERIES ERJ -> (none); SIZE / DIMENSION 0.079" L x 0.049" W (2.00mm x 1.25mm) -> (none); SUPPLIER DEVICE PACKAGE 0805 -> (none); TEMPERATURE COEFFICIENT ±100ppm/°C -> (none); TOLERANCE ±1% -> (none); UNIT PRICE (USD) 0.00729 -> (none)
- R4: @ QTY 1500 -> (none); ALTIUM_VALUE 51 -> (none); COMPOSITION Thick Film -> (none); DATASHEETS http://industrial.panasonic.com/www-cgi/jvcr13pz.cgi?E+PZ+3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 -> (none); DIGI-KEY PART NUMBER P51ACT-ND -> (none); FACTORY STOCK 0 -> (none); FAILURE RATE - -> (none); FEATURES Automotive AEC-Q200 -> (none); HEIGHT - SEATED (MAX) 0.028" (0.70mm) -> (none); IMAGE //media.digikey.com/Renders/Panasonic%20Renders/ERJ-0805%20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 -> (none); MANUFACTURER Panasonic Electronic Components -> (none); MINIMUM QUANTITY 1 -> (none); NUMBER OF TERMINATIONS 2 -> (none); OPERATING TEMPERATURE -55°C ~ 155°C -> (none); PACKAGE / CASE 0805 (2012 Metric) -> (none); PACKAGING Cut Tape (CT) -> (none); PART NUMBER ERJ-6GEYJ510V -> (none); PART STATUS Active -> (none); POWER (WATTS) 0.125W, 1/8W -> (none); Part Number (none) -> ERJ-6GEYJ510V; QUANTITY AVAILABLE 280102 -> (none); SERIES ERJ -> (none); SIZE / DIMENSION 0.079" L x 0.049" W (2.00mm x 1.25mm) -> (none); SUPPLIER DEVICE PACKAGE 0805 -> (none); TEMPERATURE COEFFICIENT ±200ppm/°C -> (none); TOLERANCE ±5% -> (none); UNIT PRICE (USD) 0.00496 -> (none)
- U1: COPYRIGHT Copyright (C) 2022 Ultra Librarian. All rights reserved. -> (none); DIGI-KEY_PART_NUMBER_1 QS6J11CT-ND -> (none); DIGI-KEY_PART_NUMBER_2 QS6J11DKR-ND -> (none); DIGI-KEY_PART_NUMBER_3 QS6J11TR-ND -> (none); MANUFACTURER_PART_NUMBER QS6J11TR -> (none); MFR_NAME ROHM Semiconductor -> (none); Part Number (none) -> QS6J11TR; REFDES RefDes -> (none); TYPE DEV -> (none)
